File: BC660K_Power.kicad_sch (KiCad schematic)
At the start: 7 parts, among them U1 BC660K

Commit message: Updated title blocks for all sheets
Other:
- company: (none) -> By AxioPaladin
- title: (none) -> BC660K Breakout Board (Power Supply)
Changed lines of the file:
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@@
 (kicad_sch (version 20211123) (generator eeschema)
-  (paper "A4")
+  (paper "USLetter")
+  (title_block
+    (title "BC660K Breakout Board (Power Supply)")
+    (date "2022-10-31")
+    (rev "X01")
+    (company "By AxioPaladin")
+    (comment 1 "CERN-OHL-W")
+  )
   (junction (at 109.22 76.2) (diameter 0) (color 0 0 0 0)
   )
