File: BC660K_SIM.kicad_sch (KiCad schematic)
At the start: 13 parts, among them J2 NanoSIM_1042240820, U1 BC660K

Commit message: Updated title blocks for all sheets
Other:
- company: (none) -> By AxioPaladin
Changed lines of the file:
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@@
     (date "2022-10-31")
     (rev "X01")
+    (company "By AxioPaladin")
+    (comment 1 "CERN-OHL-W")
   )
   (junction (at 93.98 78.74) (diameter 0) (color 0 0 0 0)
